Commit message: Correct straight driving and record wheel calibration

File: see_sys_robot_encoder/ros2_ws/src/robot_base_driver/urdf/robot_base.urdf.xacro (robot description, xacro)
@@ -12,5 +12,5 @@
 -->
 <robot name="robot_base" xmlns:xacro="http://www.ros.org/wiki/xacro">
-  <xacro:property name="wheel_radius" value="0.022" />
+  <xacro:property name="wheel_radius" value="0.021961" />
   <xacro:property name="wheel_width" value="0.014" />
   <xacro:property name="wheel_separation" value="0.116" />

Commit message: Add live RViz view for robot odometry

File: see_sys_robot_encoder/ros2_ws/src/robot_base_driver/urdf/robot_base.urdf.xacro (robot description, xacro)
@@ -28,4 +28,7 @@
     <color rgba="0.1 0.1 0.1 1.0" />
   </material>
+  <material name="front_red">
+    <color rgba="0.9 0.15 0.1 1.0" />
+  </material>
   <link name="base_link">
     <visual>
@@ -43,4 +46,18 @@
     </collision>
   </link>
+  <!-- A visible front marker makes heading clear from directly above. -->
+  <link name="front_marker">
+    <visual>
+      <geometry>
+        <box size="0.018 0.035 0.003" />
+      </geometry>
+      <material name="front_red" />
+    </visual>
+  </link>
+  <joint name="front_marker_joint" type="fixed">
+    <parent link="base_link" />
+    <child link="front_marker" />
+    <origin xyz="0.055 0 ${wheel_radius + body_height / 2 + 0.002}" rpy="0 0 0" />
+  </joint>
   <xacro:macro name="wheel" params="prefix y_sign">
     <link name="${prefix}_wheel">
